File: Eagle/4thLPF/4thLPF.brd (EAGLE design)
At the start: 100 x 80 mm, 22 parts, among them IC1 OPA2134P, IC2 TLE2426CP

Commit message: Update: Eagle Files
Parts:
- C5: device rcl:C050-035X075 -> rcl:C050-024X044
- C8: device rcl:C025-024X044 -> rcl:C050-024X044
- JP1, JP2: device pinhead:1X02/90 -> pinhead:1X02
- JP3: device pinhead:1X03/90 -> pinhead:1X03
- moved JP1 42.1 mm to (38.1, 6.35), turned to 270 degrees
- moved LED1 37.8 mm to (33.0, 6.35)
- moved R7 32.8 mm to (34.3, 10.2), turned to 0 degrees
- moved JP3 4.58 mm to (5.08, 20.3)
- moved JP2 3.81 mm to (5.08, 8.89)
- moved C5 2.54 mm to (35.6, 25.4), turned to 180 degrees
- moved C6 2.54 mm to (26.7, 27.9)
- moved C7 2.54 mm to (26.7, 7.62)
- moved IC2 2.54 mm to (34.3, 19.1)
- moved C8 1.27 mm to (12.7, 20.3)
- turned C3 to 90 degrees
- turned C4 to 270 degrees
- turned R6 to 270 degrees
Connections:
- net N$5: now also JP2.1, R1.1; no longer C4.2, IC1.7, R6.2
- net N$7: now also C4.2, IC1.7, R6.2; no longer JP2.1, R1.1
Changed lines of the file:
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@@
 <wire x1="0" y1="80" x2="0" y2="0" width="0" layer="20"/>
 <dimension x1="50.8" y1="38.1" x2="50.8" y2="2.54" x3="60.96" y3="20.32" textsize="1.778" layer="1"/>
+<dimension x1="40.64" y1="38.1" x2="2.54" y2="38.1" x3="21.59" y3="45.72" textsize="1.778" layer="1"/>
 </plain>
 <attributes>
@@
 <element name="C1" library="rcl" package="C050-035X075" value="" x="20.32" y="10.16" rot="R270"/>
 <element name="C2" library="rcl" package="C050-035X075" value="" x="15.24" y="10.16" rot="R90"/>
-<element name="C3" library="rcl" package="C050-035X075" value="" x="12.7" y="27.94" rot="R270"/>
-<element name="C4" library="rcl" package="C050-024X044" value="" x="17.78" y="27.94" rot="R90"/>
+<element name="C3" library="rcl" package="C050-035X075" value="" x="12.7" y="27.94" rot="R90"/>
+<element name="C4" library="rcl" package="C050-024X044" value="" x="17.78" y="27.94" rot="R270"/>
 <element name="IC1" library="burr-brown" package="DIL08" value="OPA2134P" x="19.05" y="19.05">
 <attribute name="OC_NEWARK" value="74K3897" x="19.05" y="19.05" size="1.778" layer="27" display="off"/>
@@
 <element name="R4" library="rcl" package="0207/7" value="" x="10.16" y="21.59" rot="R90"/>
 <element name="R5" library="rcl" package="0207/7" value="" x="20.32" y="29.21" rot="R270"/>
-<element name="R6" library="rcl" package="0207/7" value="" x="15.24" y="29.21" rot="R90"/>
-<element name="JP1" library="pinhead" package="1X02/90" value="DC-IN" x="1.27" y="26.67" rot="R90"/>
-<element name="IC2" library="tle2426" package="DIP-8" value="TLE2426CP" x="34.29" y="16.51"/>
-<element name="LED1" library="led" package="LED3MM" value="Blue" x="5.08" y="31.75" rot="R270"/>
-<element name="R7" library="rcl" package="0207/7" value="10k" x="7.62" y="29.21" rot="R270"/>
-<element name="C5" library="rcl" package="C050-035X075" value="1uF" x="38.1" y="25.4" rot="R90"/>
-<element name="C6" library="rcl" package="E2,5-6" value="10uF" x="29.21" y="27.94"/>
-<element name="C7" library="rcl" package="E2,5-6" value="10uF" x="29.21" y="7.62"/>
-<element name="JP3" library="pinhead" package="1X03/90" value="OUTPUT" x="1.27" y="17.78" rot="R90"/>
-<element name="JP2" library="pinhead" package="1X02/90" value="INPUT" x="1.27" y="8.89" rot="R90"/>
-<element name="C8" library="rcl" package="C025-024X044" value="0.1uF" x="12.7" y="21.59" rot="R270"/>
+<element name="R6" library="rcl" package="0207/7" value="" x="15.24" y="29.21" rot="R270"/>
+<element name="JP1" library="pinhead" package="1X02" value="DC-IN" x="38.1" y="6.35" rot="R270"/>
+<element name="IC2" library="tle2426" package="DIP-8" value="TLE2426CP" x="34.29" y="19.05"/>
+<element name="LED1" library="led" package="LED3MM" value="Blue" x="33.02" y="6.35" rot="R270"/>
+<element name="R7" library="rcl" package="0207/7" value="10k" x="34.29" y="10.16"/>
+<element name="C5" library="rcl" package="C050-024X044" value="1uF" x="35.56" y="25.4" rot="R180"/>
+<element name="C6" library="rcl" package="E2,5-6" value="10uF" x="26.67" y="27.94"/>
+<element name="C7" library="rcl" package="E2,5-6" value="10uF" x="26.67" y="7.62"/>
+<element name="JP3" library="pinhead" package="1X03" value="OUTPUT" x="5.08" y="20.32" rot="R90"/>
+<element name="JP2" library="pinhead" package="1X02" value="INPUT" x="5.08" y="8.89" rot="R90"/>
+<element name="C8" library="rcl" package="C050-024X044" value="0.1uF" x="12.7" y="20.32" rot="R270"/>
 <element name="C9" library="rcl" package="C025-024X044" value="0.1uF" x="25.4" y="13.97" rot="R90"/>
 </elements>
@@
 <contactref element="C8" pad="1"/>
 <contactref element="IC1" pad="8"/>
-<wire x1="30.48" y1="15.24" x2="27.94" y2="27.94" width="0" layer="19" extent="1-1"/>
-<wire x1="15.24" y1="22.86" x2="27.94" y2="27.94" width="0" layer="19" extent="1-1"/>
+<wire x1="30.48" y1="17.78" x2="25.4" y2="27.94" width="0" layer="19" extent="1-1"/>
+<wire x1="38.1" y1="10.16" x2="30.48" y2="17.78" width="0" layer="19" extent="1-1"/>
+<wire x1="38.1" y1="7.62" x2="38.1" y2="10.16" width="0" layer="19" extent="1-1"/>
+<wire x1="15.24" y1="22.86" x2="25.4" y2="27.94" width="0" layer="19" extent="1-1"/>
 <wire x1="12.7" y1="22.86" x2="15.24" y2="22.86" width="0" layer="19" extent="1-1"/>
-<wire x1="7.62" y1="25.4" x2="12.7" y2="22.86" width="0" layer="19" extent="1-1"/>
-<wire x1="5.08" y1="25.4" x2="7.62" y2="25.4" width="0" layer="19" extent="1-1"/>
 </signal>
 <signal name="V-">
@@
 <contactref element="C9" pad="2"/>
 <contactref element="IC1" pad="4"/>
-<wire x1="30.48" y1="17.78" x2="38.1" y2="27.94" width="0" layer="19" extent="1-1"/>
-<wire x1="25.4" y1="15.24" x2="30.48" y2="17.78" width="0" layer="19" extent="1-1"/>
+<wire x1="30.48" y1="20.32" x2="33.02" y2="25.4" width="0" layer="19" extent="1-1"/>
+<wire x1="25.4" y1="15.24" x2="30.48" y2="20.32" width="0" layer="19" extent="1-1"/>
 <wire x1="22.86" y1="15.24" x2="25.4" y2="15.24" width="0" layer="19" extent="1-1"/>
-<wire x1="30.48" y1="7.62" x2="25.4" y2="15.24" width="0" layer="19" extent="1-1"/>
-<wire x1="5.08" y1="27.94" x2="22.86" y2="15.24" width="0" layer="19" extent="1-1"/>
-<wire x1="5.08" y1="30.48" x2="5.08" y2="27.94" width="0" layer="19" extent="1-1"/>
+<wire x1="27.94" y1="7.62" x2="25.4" y2="15.24" width="0" layer="19" extent="1-1"/>
+<wire x1="33.02" y1="5.08" x2="27.94" y2="7.62" width="0" layer="19" extent="1-1"/>
+<wire x1="38.1" y1="5.08" x2="33.02" y2="5.08" width="0" layer="19" extent="1-1"/>
 </signal>
 <signal name="N$1">
@@
 <contactref element="C8" pad="2"/>
 <contactref element="C9" pad="1"/>
-<wire x1="30.48" y1="20.32" x2="30.48" y2="27.94" width="0" layer="19" extent="1-1"/>
-<wire x1="22.86" y1="22.86" x2="30.48" y2="20.32" width="0" layer="19" extent="1-1"/>
+<wire x1="30.48" y1="22.86" x2="27.94" y2="27.94" width="0" layer="19" extent="1-1"/>
+<wire x1="22.86" y1="22.86" x2="27.94" y2="27.94" width="0" layer="19" extent="1-1"/>
 <wire x1="20.32" y1="15.24" x2="22.86" y2="22.86" width="0" layer="19" extent="1-1"/>
 <wire x1="20.32" y1="12.7" x2="20.32" y2="15.24" width="0" layer="19" extent="1-1"/>
 <wire x1="25.4" y1="12.7" x2="20.32" y2="12.7" width="0" layer="19" extent="1-1"/>
-<wire x1="27.94" y1="7.62" x2="25.4" y2="12.7" width="0" layer="19" extent="1-1"/>
-<wire x1="12.7" y1="20.32" x2="20.32" y2="15.24" width="0" layer="19" extent="1-1"/>
-<wire x1="5.08" y1="20.32" x2="12.7" y2="20.32" width="0" layer="19" extent="1-1"/>
-<wire x1="12.7" y1="30.48" x2="12.7" y2="20.32" width="0" layer="19" extent="1-1"/>
-<wire x1="5.08" y1="10.16" x2="5.08" y2="20.32" width="0" layer="19" extent="1-1"/>
+<wire x1="25.4" y1="7.62" x2="25.4" y2="12.7" width="0" layer="19" extent="1-1"/>
+<wire x1="12.7" y1="17.78" x2="20.32" y2="15.24" width="0" layer="19" extent="1-1"/>
+<wire x1="5.08" y1="22.86" x2="12.7" y2="17.78" width="0" layer="19" extent="1-1"/>
+<wire x1="12.7" y1="25.4" x2="12.7" y2="17.78" width="0" layer="19" extent="1-1"/>
+<wire x1="5.08" y1="10.16" x2="5.08" y2="22.86" width="0" layer="19" extent="1-1"/>
 </signal>
 <signal name="N$4">
@@
 <contactref element="C3" pad="2"/>
 <contactref element="R6" pad="1"/>
-<wire x1="15.24" y1="25.4" x2="20.32" y2="33.02" width="0" layer="19" extent="1-1"/>
-<wire x1="12.7" y1="25.4" x2="15.24" y2="25.4" width="0" layer="19" extent="1-1"/>
-<wire x1="10.16" y1="25.4" x2="12.7" y2="25.4" width="0" layer="19" extent="1-1"/>
+<wire x1="15.24" y1="33.02" x2="20.32" y2="33.02" width="0" layer="19" extent="1-1"/>
+<wire x1="12.7" y1="30.48" x2="15.24" y2="33.02" width="0" layer="19" extent="1-1"/>
+<wire x1="10.16" y1="25.4" x2="12.7" y2="30.48" width="0" layer="19" extent="1-1"/>
 </signal>
 <signal name="N$3">
@@
 <contactref element="C4" pad="1"/>
 <wire x1="20.32" y1="22.86" x2="20.32" y2="25.4" width="0" layer="19" extent="1-1"/>
-<wire x1="17.78" y1="25.4" x2="20.32" y2="25.4" width="0" layer="19" extent="1-1"/>
+<wire x1="17.78" y1="30.48" x2="20.32" y2="25.4" width="0" layer="19" extent="1-1"/>
 </signal>
 <signal name="N$5">
-<contactref element="IC1" pad="7"/>
-<contactref element="R6" pad="2"/>
-<contactref element="C4" pad="2"/>
+<contactref element="JP2" pad="1"/>
+<contactref element="R1" pad="1"/>
 <contactref element="JP3" pad="1"/>
-<wire x1="17.78" y1="30.48" x2="15.24" y2="33.02" width="0" layer="19" extent="1-1"/>
-<wire x1="17.78" y1="22.86" x2="17.78" y2="30.48" width="0" layer="19" extent="1-1"/>
-<wire x1="5.08" y1="15.24" x2="17.78" y2="22.86" width="0" layer="19" extent="1-1"/>
+<wire x1="5.08" y1="17.78" x2="12.7" y2="12.7" width="0" layer="19" extent="1-1"/>
+<wire x1="5.08" y1="7.62" x2="12.7" y2="12.7" width="0" layer="19" extent="1-1"/>
 </signal>
 <signal name="N$9">
 <contactref element="R7" pad="1"/>
 <contactref element="LED1" pad="A"/>
-<wire x1="5.08" y1="33.02" x2="7.62" y2="33.02" width="0" layer="19" extent="1-1"/>
+<wire x1="33.02" y1="7.62" x2="30.48" y2="10.16" width="0" layer="19" extent="1-1"/>
 </signal>
 <signal name="N$8">
 <contactref element="IC2" pad="8"/>
 <contactref element="C5" pad="1"/>
-<wire x1="38.1" y1="20.32" x2="38.1" y2="22.86" width="0" layer="19" extent="1-1"/>
+<wire x1="38.1" y1="22.86" x2="38.1" y2="25.4" width="0" layer="19" extent="1-1"/>
 </signal>
 <signal name="N$7">
-<contactref element="R1" pad="1"/>
-<contactref element="JP2" pad="1"/>
 <contactref element="JP3" pad="2"/>
-<wire x1="5.08" y1="17.78" x2="12.7" y2="12.7" width="0" layer="19" extent="1-1"/>
-<wire x1="5.08" y1="7.62" x2="12.7" y2="12.7" width="0" layer="19" extent="1-1"/>
+<contactref element="C4" pad="2"/>
+<contactref element="IC1" pad="7"/>
+<contactref element="R6" pad="2"/>
+<wire x1="15.24" y1="25.4" x2="17.78" y2="25.4" width="0" layer="19" extent="1-1"/>
+<wire x1="17.78" y1="22.86" x2="17.78" y2="25.4" width="0" layer="19" extent="1-1"/>
+<wire x1="5.08" y1="20.32" x2="17.78" y2="22.86" width="0" layer="19" extent="1-1"/>
 </signal>
 </signals>

Commit message: 基板図作成
Parts:
- C1, C3: value (none) -> 560p
- C2: value (none) -> 100p
- C4: value (none) -> 10p
- C6, C7: value 10uF -> 100uF
- IC1: value OPA2134P -> NJM2068
- R1, R3: value (none) -> 2.7k
- R2: value (none) -> 6.8k
- R4, R6: value (none) -> 7.5k
- R5: value (none) -> 12k
- moved C5 2.54 mm to (35.6, 27.9)
- moved C9 2.54 mm to (25.4, 16.5)
- moved JP1 2.54 mm to (38.1, 8.89)
- moved LED1 2.54 mm to (33.0, 8.89)
- moved C7 2.54 mm to (26.7, 10.2)
- moved C1 2.54 mm to (20.3, 12.7)
- moved C2 2.54 mm to (15.2, 12.7)
- moved C3 2.54 mm to (12.7, 30.5)
- moved C4 2.54 mm to (17.8, 30.5)
- moved C6 2.54 mm to (26.7, 30.5)
- moved C8 2.54 mm to (12.7, 22.9)
- moved IC1 2.54 mm to (19.1, 21.6)
- moved IC2 2.54 mm to (34.3, 21.6)
- moved JP2 2.54 mm to (5.08, 11.4)
- moved JP3 2.54 mm to (5.08, 22.9)
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Routing:
- net GND: track 0.00 -> 109.8 mm
- net V+: track 0.00 -> 61.6 mm
- net V-: track 0.00 -> 39.2 mm
- net N$5: track 0.00 -> 23.9 mm
- net N$7: track 0.00 -> 20.3 mm
- net N$6: track 0.00 -> 20.3 mm
- net N$4: track 0.00 -> 12.7 mm
- net N$1: track 0.00 -> 11.2 mm
- net N$3: track 0.00 -> 8.67 mm
- net N$2: track 0.00 -> 8.67 mm
- net N$9: track 0.00 -> 3.59 mm
- net N$8: track 0.00 -> 2.54 mm
Other:
- board size 100 x 80 mm -> 42.9 x 40.6 mm
