File: Eagle/4thLPF/4thLPF.sch (EAGLE design)
At the start: 22 parts, among them IC1 OPA2134P, IC2 TLE2426CP

Commit message: Update: Eagle Files
Parts:
- C5: device rcl:C-EU050-035X075 -> rcl:C-EU050-024X044
- C8: device rcl:C-EU025-024X044 -> rcl:C-EU050-024X044
- JP1, JP2: device pinhead:PINHD-1X2/90 -> pinhead:PINHD-1X2
- JP3: device pinhead:PINHD-1X3/90 -> pinhead:PINHD-1X3
Connections:
- net N$5: now also JP2.1, R1.1; no longer C4.2, IC1B.OUT, R6.2
- net N$7: now also C4.2, IC1B.OUT, R6.2; no longer JP2.1, R1.1
Other:
- moved on the sheet: JP3
Changed lines of the file:
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@@
 <setting verticaltext="up"/>
 </settings>
-<grid distance="0.1" unitdist="inch" unit="inch" style="dots" multiple="1" display="yes" altdistance="0.01" altunitdist="inch" altunit="inch"/>
+<grid distance="0.1" unitdist="inch" unit="inch" style="lines" multiple="1" display="no" altdistance="0.01" altunitdist="inch" altunit="inch"/>
 <layers>
 <layer number="1" name="Top" color="4" fill="1" visible="no" active="no"/>
@@
 <part name="GND5" library="supply1" deviceset="GND" device=""/>
 <part name="GND6" library="supply1" deviceset="GND" device=""/>
-<part name="JP1" library="pinhead" deviceset="PINHD-1X2" device="/90" value="DC-IN"/>
+<part name="JP1" library="pinhead" deviceset="PINHD-1X2" device="" value="DC-IN"/>
 <part name="P-1" library="supply1" deviceset="V-" device=""/>
 <part name="P+1" library="supply1" deviceset="V+" device=""/>
@@
 <part name="LED1" library="led" deviceset="LED" device="3MM" value="Blue"/>
 <part name="R7" library="rcl" deviceset="R-EU_" device="0207/7" value="10k"/>
-<part name="C5" library="rcl" deviceset="C-EU" device="050-035X075" value="1uF"/>
+<part name="C5" library="rcl" deviceset="C-EU" device="050-024X044" value="1uF"/>
 <part name="C6" library="rcl" deviceset="CPOL-EU" device="E2.5-6" value="10uF"/>
 <part name="C7" library="rcl" deviceset="CPOL-EU" device="E2.5-6" value="10uF"/>
-<part name="JP3" library="pinhead" deviceset="PINHD-1X3" device="/90" value="OUTPUT"/>
-<part name="JP2" library="pinhead" deviceset="PINHD-1X2" device="/90" value="INPUT"/>
+<part name="JP3" library="pinhead" deviceset="PINHD-1X3" device="" value="OUTPUT"/>
+<part name="JP2" library="pinhead" deviceset="PINHD-1X2" device="" value="INPUT"/>
 <part name="P+2" library="supply1" deviceset="V+" device=""/>
 <part name="P-2" library="supply1" deviceset="V-" device=""/>
-<part name="C8" library="rcl" deviceset="C-EU" device="025-024X044" value="0.1uF"/>
+<part name="C8" library="rcl" deviceset="C-EU" device="050-024X044" value="0.1uF"/>
 <part name="C9" library="rcl" deviceset="C-EU" device="025-024X044" value="0.1uF"/>
 </parts>
@@
 <instance part="C6" gate="G$1" x="43.18" y="132.08"/>
 <instance part="C7" gate="G$1" x="43.18" y="119.38"/>
-<instance part="JP3" gate="A" x="127" y="50.8"/>
+<instance part="JP3" gate="A" x="127" y="53.34"/>
 <instance part="JP2" gate="G$1" x="-15.24" y="55.88" rot="MR0"/>
 <instance part="P+2" gate="1" x="38.1" y="43.18" rot="R180"/>
@@
 <segment>
 <pinref part="GND6" gate="1" pin="GND"/>
-<wire x1="106.68" y1="40.64" x2="106.68" y2="48.26" width="0.1524" layer="91"/>
+<wire x1="106.68" y1="40.64" x2="106.68" y2="50.8" width="0.1524" layer="91"/>
 <pinref part="JP3" gate="A" pin="3"/>
-<wire x1="124.46" y1="48.26" x2="106.68" y2="48.26" width="0.1524" layer="91"/>
+<wire x1="124.46" y1="50.8" x2="106.68" y2="50.8" width="0.1524" layer="91"/>
 </segment>
 <segment>
@@
 <net name="N$5" class="0">
 <segment>
-<pinref part="IC1" gate="B" pin="OUT"/>
-<wire x1="101.6" y1="53.34" x2="106.68" y2="53.34" width="0.1524" layer="91"/>
-<pinref part="R6" gate="G$1" pin="2"/>
-<wire x1="106.68" y1="53.34" x2="106.68" y2="78.74" width="0.1524" layer="91"/>
-<wire x1="106.68" y1="78.74" x2="83.82" y2="78.74" width="0.1524" layer="91"/>
-<pinref part="C4" gate="G$1" pin="2"/>
-<wire x1="83.82" y1="78.74" x2="81.28" y2="78.74" width="0.1524" layer="91"/>
-<wire x1="83.82" y1="71.12" x2="83.82" y2="78.74" width="0.1524" layer="91"/>
-<junction x="83.82" y="78.74"/>
+<wire x1="-2.54" y1="86.36" x2="114.3" y2="86.36" width="0.1524" layer="91"/>
+<wire x1="114.3" y1="86.36" x2="114.3" y2="55.88" width="0.1524" layer="91"/>
+<pinref part="R1" gate="G$1" pin="1"/>
+<pinref part="JP2" gate="G$1" pin="1"/>
+<wire x1="-12.7" y1="58.42" x2="-2.54" y2="58.42" width="0.1524" layer="91"/>
+<wire x1="-2.54" y1="58.42" x2="0" y2="58.42" width="0.1524" layer="91"/>
+<wire x1="-2.54" y1="86.36" x2="-2.54" y2="58.42" width="0.1524" layer="91"/>
+<junction x="-2.54" y="58.42"/>
 <pinref part="JP3" gate="A" pin="1"/>
-<wire x1="124.46" y1="53.34" x2="106.68" y2="53.34" width="0.1524" layer="91"/>
-<junction x="106.68" y="53.34"/>
+<wire x1="124.46" y1="55.88" x2="114.3" y2="55.88" width="0.1524" layer="91"/>
 </segment>
 </net>
@@
 <net name="N$7" class="0">
 <segment>
-<wire x1="-2.54" y1="86.36" x2="114.3" y2="86.36" width="0.1524" layer="91"/>
-<wire x1="114.3" y1="86.36" x2="114.3" y2="50.8" width="0.1524" layer="91"/>
-<pinref part="R1" gate="G$1" pin="1"/>
-<pinref part="JP2" gate="G$1" pin="1"/>
-<wire x1="-12.7" y1="58.42" x2="-2.54" y2="58.42" width="0.1524" layer="91"/>
-<wire x1="-2.54" y1="58.42" x2="0" y2="58.42" width="0.1524" layer="91"/>
-<wire x1="-2.54" y1="86.36" x2="-2.54" y2="58.42" width="0.1524" layer="91"/>
-<junction x="-2.54" y="58.42"/>
+<pinref part="R6" gate="G$1" pin="2"/>
 <pinref part="JP3" gate="A" pin="2"/>
-<wire x1="114.3" y1="50.8" x2="124.46" y2="50.8" width="0.1524" layer="91"/>
-</segment>
-</net>
+<pinref part="IC1" gate="B" pin="OUT"/>
+<wire x1="101.6" y1="53.34" x2="106.68" y2="53.34" width="0.1524" layer="91"/>
+<wire x1="106.68" y1="53.34" x2="124.46" y2="53.34" width="0.1524" layer="91"/>
+<junction x="106.68" y="53.34"/>
+<wire x1="106.68" y1="53.34" x2="106.68" y2="78.74" width="0.1524" layer="91"/>
+<wire x1="106.68" y1="78.74" x2="83.82" y2="78.74" width="0.1524" layer="91"/>
+<wire x1="83.82" y1="78.74" x2="81.28" y2="78.74" width="0.1524" layer="91"/>
+<junction x="83.82" y="78.74"/>
+<pinref part="C4" gate="G$1" pin="2"/>
+<wire x1="83.82" y1="71.12" x2="83.82" y2="78.74" width="0.1524" layer="91"/>
+</segment>
+</net>

Commit message: 基板図作成
Parts:
- C1, C3: value (none) -> 560p
- C2: value (none) -> 100p
- C4: value (none) -> 10p
- C6, C7: value 10uF -> 100uF
- IC1: value OPA2134P -> NJM2068
- R1, R3: value (none) -> 2.7k
- R2: value (none) -> 6.8k
- R4, R6: value (none) -> 7.5k
- R5: value (none) -> 12k
Changed lines of the file:
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@@
 <setting verticaltext="up"/>
 </settings>
-<grid distance="0.1" unitdist="inch" unit="inch" style="lines" multiple="1" display="no" altdistance="0.01" altunitdist="inch" altunit="inch"/>
+<grid distance="0.1" unitdist="inch" unit="inch" style="lines" multiple="1" display="yes" altdistance="0.01" altunitdist="inch" altunit="inch"/>
 <layers>
 <layer number="1" name="Top" color="4" fill="1" visible="no" active="no"/>
@@
 </classes>
 <parts>
-<part name="IC1" library="burr-brown" deviceset="OPA2134" device="P"/>
+<part name="IC1" library="burr-brown" deviceset="OPA2134" device="P" value="NJM2068"/>
 <part name="GND1" library="supply1" deviceset="GND" device=""/>
-<part name="R1" library="rcl" deviceset="R-EU_" device="0207/7"/>
-<part name="C1" library="rcl" deviceset="C-EU" device="050-035X075"/>
-<part name="C2" library="rcl" deviceset="C-EU" device="050-035X075"/>
-<part name="R2" library="rcl" deviceset="R-EU_" device="0207/7"/>
-<part name="R3" library="rcl" deviceset="R-EU_" device="0207/7"/>
+<part name="R1" library="rcl" deviceset="R-EU_" device="0207/7" value="2.7k"/>
+<part name="C1" library="rcl" deviceset="C-EU" device="050-035X075" value="560p"/>
+<part name="C2" library="rcl" deviceset="C-EU" device="050-035X075" value="100p"/>
+<part name="R2" library="rcl" deviceset="R-EU_" device="0207/7" value="6.8k"/>
+<part name="R3" library="rcl" deviceset="R-EU_" device="0207/7" value="2.7k"/>
 <part name="GND2" library="supply1" deviceset="GND" device=""/>
-<part name="R4" library="rcl" deviceset="R-EU_" device="0207/7"/>
-<part name="R5" library="rcl" deviceset="R-EU_" device="0207/7"/>
-<part name="R6" library="rcl" deviceset="R-EU_" device="0207/7"/>
-<part name="C3" library="rcl" deviceset="C-EU" device="050-035X075"/>
-<part name="C4" library="rcl" deviceset="C-EU" device="050-024X044"/>
+<part name="R4" library="rcl" deviceset="R-EU_" device="0207/7" value="7.5k"/>
+<part name="R5" library="rcl" deviceset="R-EU_" device="0207/7" value="12k"/>
+<part name="R6" library="rcl" deviceset="R-EU_" device="0207/7" value="7.5k"/>
+<part name="C3" library="rcl" deviceset="C-EU" device="050-035X075" value="560p"/>
+<part name="C4" library="rcl" deviceset="C-EU" device="050-024X044" value="10p"/>
 <part name="GND3" library="supply1" deviceset="GND" device=""/>
 <part name="GND4" library="supply1" deviceset="GND" device=""/>
@@
 <part name="R7" library="rcl" deviceset="R-EU_" device="0207/7" value="10k"/>
 <part name="C5" library="rcl" deviceset="C-EU" device="050-024X044" value="1uF"/>
-<part name="C6" library="rcl" deviceset="CPOL-EU" device="E2.5-6" value="10uF"/>
-<part name="C7" library="rcl" deviceset="CPOL-EU" device="E2.5-6" value="10uF"/>
+<part name="C6" library="rcl" deviceset="CPOL-EU" device="E2.5-6" value="100uF"/>
+<part name="C7" library="rcl" deviceset="CPOL-EU" device="E2.5-6" value="100uF"/>
 <part name="JP3" library="pinhead" deviceset="PINHD-1X3" device="" value="OUTPUT"/>
 <part name="JP2" library="pinhead" deviceset="PINHD-1X2" device="" value="INPUT"/>
